File: src/kicad/Devboard.kicad_pcb (KiCad board)
At the start: 4 copper layers, 48 x 37 mm, 49 parts, among them J1 USB_C_Receptacle_USB2.0_16P, J2 Conn_01x06, J3 Conn_01x06, J4 Conn_01x02, SW1 RESET, SW2 BOOT, U1 XC6220B331MR, U2 ESP32-C3, U3 W25Q128JVS, Y1 40MHz

Commit message: Update Journal
Parts:
- C1: value 47uF -> 10uF
- C10, C13, C3, C4, C5, C6, C7, C9: footprint Capacitor_SMD:C_0603_1608Metric -> Capacitor_SMD:C_0201_0603Metric
- C2: value 47uF -> 4.7uF; footprint Capacitor_SMD:C_0603_1608Metric -> Capacitor_SMD:C_0201_0603Metric
- R10, R11, R12, R7, R8, R9: value 0 -> 22
- moved C1 35.9 mm to (180.2, 100.1)
- moved C2 35.9 mm to (183.4, 104.5)
- moved U1 35.9 mm to (180.2, 103.9)
- moved D3 29.8 mm to (176.0, 79.5), turned to -90 degrees
- moved D2 29.4 mm to (173.0, 79.5), turned to -90 degrees
- moved R6 23.5 mm to (176.0, 82.7), turned to -90 degrees
- moved J2 22.6 mm to (179.0, 110.0), turned to -90 degrees
- moved R5 22.1 mm to (173.0, 83.2), turned to -90 degrees
- moved L1 14.0 mm to (165.0, 99.0), turned to 0 degrees
- moved C9 13.6 mm to (165.0, 98.0), turned to 180 degrees
- moved C13 11.5 mm to (167.2, 87.0), turned to 180 degrees
- moved AE1 10.8 mm to (182.0, 89.0), turned to 0 degrees
- moved C11 10.0 mm to (174.0, 106.0)
- moved L3 8.94 mm to (176.0, 91.0), turned to 45 degrees
- moved C14 8.79 mm to (175.0, 91.5), turned to -45 degrees
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Connections:
- C1 pad 1: VCC -> VBUS
- C2 pad 1: VCC -> +3V3
- J3 pad 2: /GPIO9 -> /GPIO8
- R4 pad 1: /GPIO8 -> /GPIO9
- SW2 pad 1: /GPIO8 -> /GPIO9
- SW2 pad 2: +3V3 -> GND
- U1 pad 1: VCC -> VBUS
- U1 pad 3: VCC -> VBUS
- U1 pad 5: VCC -> +3V3
Routing:
- net +3V3: track 38.8 -> 16.2 mm, vias 1 -> 0
- net GND: track 52.2 -> 33.0 mm, vias 26 -> 31
- net /CHIP_EN: track 23.6 -> 41.0 mm, vias 2 -> 1
- net VBUS: track 40.9 -> 57.1 mm, vias 3 -> 2
- net VCC: track 11.4 -> 0.00 mm
- net +3.3V: track 48.2 -> 38.3 mm
- net /GPIO4: track 23.7 -> 15.0 mm, vias 2 -> 0
- net Net-(C12-Pad1): track 5.38 -> 12.2 mm
- net Net-(U2-XTAL_N): track 11.3 -> 17.3 mm
- net Net-(C10-Pad1): track 23.8 -> 18.5 mm, vias 0 -> 2
- net /GPIO8: track 9.96 -> 14.2 mm, vias 2 -> 0
- net /GPIO1: track 21.7 -> 25.5 mm, vias 2 -> 1
- net /GPIO9: track 14.0 -> 11.0 mm, vias 1 -> 0
- net /RXD: track 11.4 -> 13.8 mm
- net Net-(AE1-FEED): track 7.08 -> 5.06 mm
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Other:
- board text added: "8"
- board text removed: "9"

Commit message: Update Journal after review
Parts:
- C10, C13, C2, C3, C4, C5, C6, C7, C9: footprint Capacitor_SMD:C_0201_0603Metric -> Capacitor_SMD:C_0402_1005Metric
- L1, L2: footprint Inductor_SMD:L_0201_0603Metric -> Inductor_SMD:L_0402_1005Metric
- R1, R10, R11, R12, R13, R2, R3, R4, R5, R6, R7, R8, R9: footprint Resistor_SMD:R_0201_0603Metric -> Resistor_SMD:R_0603_1608Metric
- moved R12 3.34 mm to (155.0, 100.0), turned to 45 degrees
- moved AE1 3.00 mm to (185.0, 89.0), turned to -90 degrees
- moved R7 2.15 mm to (155.5, 91.4)
- moved R6 2.02 mm to (178.0, 83.0)
- moved R5 2.01 mm to (175.0, 83.0)
- moved D2 2.00 mm to (175.0, 79.5)
- moved D3 2.00 mm to (178.0, 79.5)
- moved R1 1.83 mm to (155.0, 103.0), turned to -135 degrees
- moved R11 1.82 mm to (155.3, 97.5)
- moved C5 1.61 mm to (157.0, 89.7)
- moved R8 1.41 mm to (156.0, 93.0)
- moved R9 1.12 mm to (156.0, 94.5)
- moved L2 1.00 mm to (163.0, 100.0)
- moved R10 1.00 mm to (156.0, 96.0)
- moved R2 0.11 mm to (150.0, 104.0)
Routing:
- net Net-(AE1-FEED): track 5.06 -> 10.1 mm
- net Net-(U2-SPIQ): track 2.24 -> 5.01 mm
- net /SPID: track 7.13 -> 5.10 mm
- net /SPIQ: track 16.8 -> 14.9 mm
- net /GPIO4: track 15.0 -> 16.9 mm
- net /GPIO2: track 16.3 -> 18.0 mm
- net Net-(U2-SPIHD): track 2.31 -> 3.94 mm
- net /VDD_SPI: track 11.3 -> 12.9 mm
- net /SPICS0: track 15.4 -> 13.8 mm
- net /SPICLK: track 7.24 -> 5.74 mm
- net Net-(U2-SPID): track 2.48 -> 3.93 mm
- net /SPICHD: track 7.66 -> 6.31 mm
- net /SPICWP: track 14.9 -> 13.9 mm
- net Net-(J1-CC2): track 1.96 -> 2.95 mm
- net Net-(U2-SPIWP): track 2.10 -> 3.01 mm
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
Commit message: Update project
Parts:
- C2: footprint Capacitor_SMD:C_0402_1005Metric -> Capacitor_SMD:C_0603_1608Metric
- moved H1 2.24 mm to (143.0, 81.0)
- moved H2 2.00 mm to (184.0, 81.0)
- moved D2 1.71 mm to (175.0, 81.2)
- moved D3 1.71 mm to (178.0, 81.2)
- moved R5 1.71 mm to (175.0, 84.7)
- moved R6 1.71 mm to (178.0, 84.7)
- moved H3 1.00 mm to (143.0, 110.0)
- moved J3 1.00 mm to (155.9, 80.0)
Routing:
- net /GPIO8: track 14.2 -> 13.2 mm
- net /GPIO6: track 13.7 -> 12.7 mm
- net /GPIO5: track 14.4 -> 13.4 mm
- net /GPIO3: track 15.6 -> 14.6 mm
- net /GPIO10: track 14.8 -> 13.8 mm
- net /GPIO2: track 18.0 -> 17.2 mm
- net /GPIO4: track 16.9 -> 16.2 mm
Other:
- board size 48 x 37 mm -> 47 x 35 mm

Commit message: Update project
Parts:
- C11, C12: value 10uF -> 10pF
- turned R4 to 90 degrees
Connections:
- R4 pad 1: /GPIO9 -> +3.3V
- R4 pad 2: GND -> /GPIO9
Routing:
- net GND: track 33.2 -> 31.7 mm, vias 31 -> 30
- net +3.3V: track 38.5 -> 39.7 mm
- net /GPIO7: track 13.3 -> 12.3 mm
- net /GPIO0: track 24.1 -> 23.2 mm
Changed lines of the file:
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@@
 			)
 		)
-		(property "Value" "10uF"
+		(property "Value" "10pF"
 			(at 0 1.43 0)
 			(layer "F.Fab")
@@
 			)
 		)
-		(property "LCSC Part" "C96446"
+		(property "LCSC Part" "C1634"
 			(at 0 0 0)
 			(unlocked yes)
@@
 		(model "${EASYEDA2KICAD}/easyeda2kicad.3dshapes/USB-C-SMD_TYPE-C-6PIN-2MD-073.wrl"
 			(offset
-				(xyz 0 0 0)
+				(xyz 0 -1.5 1.5)
 			)
 			(scale
@@
 			)
 			(rotate
-				(xyz 0 0 0)
+				(xyz -0 -0 -0)
 			)
 		)
@@
 	(footprint "Resistor_SMD:R_0603_1608Metric"
 		(layer "F.Cu")
-		(at 155.82 87 -90)
+		(at 155.82 87 90)
 		(descr "Resistor SMD 0603 (1608 Metric), square (rectangular) end terminal, IPC-7351 nominal, (Body size source: IPC-SM-782 page 72, https://www.pcb-3d.com/wordpress/wp-content/uploads/ipc-sm-782a_amendment_1_and_2.pdf)")
 		(tags "resistor")
 		(property "Reference" "R4"
-			(at 0 -1.43 270)
+			(at 0 -1.43 90)
 			(layer "F.SilkS")
 			(hide yes)
@@
 		)
 		(property "Value" "10k"
-			(at 0 1.43 270)
+			(at 0 1.43 90)
 			(layer "F.Fab")
 			(effects
@@
 		)
 		(property "Datasheet" ""
-			(at 0 0 270)
+			(at 0 0 90)
 			(layer "F.Fab")
 			(hide yes)
@@
 		)
 		(property "Description" "Resistor"
-			(at 0 0 270)
+			(at 0 0 90)
 			(layer "F.Fab")
 			(hide yes)
@@
 		)
 		(property "KiLib_Generator" "SMD_2terminal_chip_molded"
-			(at 0 0 270)
+			(at 0 0 90)
 			(layer "F.SilkS")
 			(hide yes)
@@
 		)
 		(property "LCSC Part" "C2930027"
-			(at 0 0 270)
+			(at 0 0 90)
 			(unlocked yes)
 			(layer "F.Fab")
@@
 		)
 		(property "KLC_S3.3" ""
-			(at 0 0 270)
+			(at 0 0 90)
 			(unlocked yes)
 			(layer "F.Fab")
@@
 		)
 		(property "KLC_S4.1" ""
-			(at 0 0 270)
+			(at 0 0 90)
 			(unlocked yes)
 			(layer "F.Fab")
@@
 		(duplicate_pad_numbers_are_jumpers no)
 		(fp_line
-			(start -0.237258 0.5225)
-			(end 0.237258 0.5225)
+			(start -0.237258 -0.5225)
+			(end 0.237258 -0.5225)
 			(stroke
 				(width 0.12)
@@
 		)
 		(fp_line
-			(start -0.237258 -0.5225)
-			(end 0.237258 -0.5225)
+			(start -0.237258 0.5225)
+			(end 0.237258 0.5225)
 			(stroke
 				(width 0.12)
@@
 		)
 		(fp_text user "${REFERENCE}"
-			(at 0 0 270)
+			(at 0 0 90)
 			(layer "F.Fab")
 			(effects
@@
 		)
 		(pad "1" smd roundrect
-			(at -0.825 0 270)
+			(at -0.825 0 90)
 			(size 0.8 0.95)
 			(layers "F.Cu" "F.Mask" "F.Paste")
 			(roundrect_rratio 0.25)
-			(net "/GPIO9")
+			(net "+3.3V")
 			(pintype "passive")
 		)
 		(pad "2" smd roundrect
-			(at 0.825 0 270)
+			(at 0.825 0 90)
 			(size 0.8 0.95)
 			(layers "F.Cu" "F.Mask" "F.Paste")
 			(roundrect_rratio 0.25)
-			(net "GND")
+			(net "/GPIO9")
 			(pintype "passive")
 		)
@@
 			)
 		)
-		(property "Value" "10uF"
+		(property "Value" "10pF"
 			(at 0 1.43 0)
 			(layer "F.Fab")
@@
 			)
 		)
-		(property "LCSC Part" "C96446"
+		(property "LCSC Part" "C1634"
 			(at 0 0 0)
 			(unlocked yes)
@@
 			)
 		)
-		(property "LCSC Part" "C23733"
+		(property "LCSC Part" "C69335"
 			(at 0 0 270)
 			(unlocked yes)
@@
 	)
 	(segment
-		(start 155.82 87.825)
-		(end 155.82 88.18)
-		(width 0.2)
-		(layer "F.Cu")
-		(net "GND")
-	)
-	(segment
 		(start 177.1625 104.725)
 		(end 177.1625 106.3625)
@@
 	)
 	(segment
-		(start 155.82 88.18)
-		(end 155 89)
-		(width 0.2)
-		(layer "F.Cu")
-		(net "GND")
-	)
-	(segment
 		(start 158 87.68)
 		(end 158.68 87.68)
@@
 	)
 	(via
-		(at 155 89)
-		(size 0.6)
-		(drill 0.3)
-		(layers "F.Cu" "B.Cu")
-		(net "GND")
-	)
-	(via
 		(at 160 87)
 		(size 0.6)
@@
 	)
 	(segment
+		(start 155.82 87.825)
+		(end 156.825 87.825)
+		(width 0.2)
+		(layer "F.Cu")
+		(net "+3.3V")
+	)
+	(segment
 		(start 163.93 90.07)
 		(end 164 90)
@@
 	)
 	(segment
+		(start 156.825 87.825)
+		(end 157 88)
+		(width 0.2)
+		(layer "F.Cu")
+		(net "+3.3V")
+	)
+	(segment
 		(start 158 92)
 		(end 158 88.32)
@@
 	)
 	(segment
-		(start 168 110)
-		(end 168.84 110)
-		(width 0.2)
-		(layer "B.Cu")
-		(net "/GPIO0")
-	)
-	(segment
 		(start 168.84 108.082893)
 		(end 168.84 110)
@@
 	)
 	(segment
-		(start 161.5 80.5)
-		(end 161 80)
+		(start 161 80)
+		(end 161.5 80.5)
 		(width 0.2)
 		(layer "F.Cu")
@@
 	)
 	(segment
-		(start 161.5 92.1)
-		(end 161.5 79.5)
+		(start 161.5 80.5)
+		(end 161.5 92.1)
 		(width 0.2)
 		(layer "F.Cu")
@@
 	)
 	(segment
-		(start 159.5 89.207107)
-		(end 159.5 87.5)
+		(start 160.5 92.1)
+		(end 160.5 90.207107)
 		(width 0.2)
 		(layer "F.Cu")
@@
 	)
 	(segment
-		(start 159.5 87.5)
-		(end 158.175 86.175)
+		(start 154.825 86.175)
+		(end 154 87)
 		(width 0.2)
 		(layer "F.Cu")
@@
 	)
 	(segment
-		(start 154 87)
-		(end 154.995 87)
+		(start 159.5 89.207107)
+		(end 159.5 87.792893)
 		(width 0.2)
 		(layer "F.Cu")
@@
 	)
 	(segment
-		(start 160.5 90.207107)
-		(end 159.5 89.207107)
+		(start 157.882107 86.175)
+		(end 155.82 86.175)
 		(width 0.2)
 		(layer "F.Cu")
@@
 	)
 	(segment
-		(start 154.995 87)
-		(end 155.82 86.175)
+		(start 155.82 86.175)
+		(end 154.825 86.175)
 		(width 0.2)
 		(layer "F.Cu")
@@
 	)
 	(segment
-		(start 160.5 92.1)
-		(end 160.5 90.207107)
+		(start 159.5 87.792893)
+		(end 157.882107 86.175)
 		(width 0.2)
 		(layer "F.Cu")
@@
 	)
 	(segment
-		(start 158.175 86.175)
-		(end 155.82 86.175)
+		(start 160.5 90.207107)
+		(end 159.5 89.207107)
 		(width 0.2)
 		(layer "F.Cu")
@@
 	)
 	(segment
-		(start 154.15 106.15)
-		(end 154.15 106.58)
-		(width 0.2)
-		(layer "F.Cu")
-		(net "VBUS")
-	)
-	(segment
 		(start 166.3 110)
 		(end 167 109.3)
@@
 	)
 	(segment
-		(start 149.95 107.18)
-		(end 149.35 106.58)
-		(width 0.2)
-		(layer "F.Cu")
-		(net "VBUS")
-	)
-	(segment
 		(start 179.512501 106.0375)
 		(end 179.2125 105.737499)
@@
 	)
 	(segment
-		(start 181.1125 105.075)
-		(end 181.1625 105.075)
+		(start 149.95 107.18)
+		(end 149.35 106.58)
 		(width 0.2)
 		(layer "F.Cu")
@@
 	)
 	(segment
-		(start 153.55 107.18)
-		(end 149.95 107.18)
+		(start 181.1125 105.075)
+		(end 181.1625 105.075)
 		(width 0.2)
 		(layer "F.Cu")
@@
 	)
 	(segment
-		(start 149.35 106.58)
-		(end 149.35 106.15)
-		(width 0.2)
-		(layer "F.Cu")
-		(net "VBUS")
-	)
-	(segment
 		(start 178.1625 101.3)
 		(end 179.3875 100.075)
@@
 	)
 	(segment
+		(start 153.55 107.18)
+		(end 149.95 107.18)
+		(width 0.2)
+		(layer "F.Cu")
+		(net "VBUS")
+	)
+	(segment
+		(start 149.35 106.58)
+		(end 149.35 106.15)
+		(width 0.2)
+		(layer "F.Cu")
+		(net "VBUS")
+	)
+	(segment
 		(start 165.26 111.04)
 		(end 166.3 110)
@@
 	)
 	(segment
+		(start 154.15 106.58)
+		(end 153.55 107.18)
+		(width 0.2)
+		(layer "F.Cu")
+		(net "VBUS")
+	)
+	(segment
 		(start 178.1625 104.025)
 		(end 178.1625 101.3)
@@
 	)
 	(segment
-		(start 154.15 106.58)
-		(end 153.55 107.18)
+		(start 154.15 106.15)
+		(end 154.15 106.58)
 		(width 0.2)
 		(layer "F.Cu")
