File: src/kicad/Devboard.kicad_sch (KiCad schematic)
At the start: 49 parts, among them J1 USB_C_Receptacle_USB2.0_16P, J2 Conn_01x06, J3 Conn_01x06, J4 Conn_01x02, SW1 RESET, SW2 BOOT, U1 XC6220B331MR, U2 ESP32-C3, U3 W25Q128JVS, Y1 40MHz

Commit message: Update Journal
Parts:
- C1: value 47uF -> 10uF; LCSC Part C140782 -> C96446
- C10, C13, C3, C5, C7: footprint Capacitor_SMD:C_0603_1608Metric -> Capacitor_SMD:C_0201_0603Metric; LCSC Part C15849 -> C76935
- C2: value 47uF -> 4.7uF; footprint Capacitor_SMD:C_0603_1608Metric -> Capacitor_SMD:C_0201_0603Metric; LCSC Part C140782 -> C47117441
- C4, C9: footprint Capacitor_SMD:C_0603_1608Metric -> Capacitor_SMD:C_0201_0603Metric; LCSC Part C15849 -> C307380
- C6: footprint Capacitor_SMD:C_0603_1608Metric -> Capacitor_SMD:C_0201_0603Metric; LCSC Part C100042 -> C272853
- R10, R11, R12, R7, R8, R9: value 0 -> 22; LCSC Part C100044 -> C23345
Connections:
- net +3V3: now also C2.1, U1.5 (VOUT); no longer SW2.2
- net GND: now also SW2.2
- net GPIO8: now also J3.2 (Pin_2); no longer R4.1, SW2.1
- net GPIO9: now also R4.1, SW2.1; no longer J3.2 (Pin_2)
- net VBUS: now also C1.1, U1.1 (VIN), U1.3 (CE)
- removed net VCC: C1.1, C2.1, U1.1 (VIN), U1.3 (CE), U1.5 (VOUT)
Other:
- moved on the sheet: C1, C2

Commit message: Update Journal after review
Parts:
- C10, C13, C3, C5, C7: footprint Capacitor_SMD:C_0201_0603Metric -> Capacitor_SMD:C_0402_1005Metric; LCSC Part C76935 -> C52923
- C2: footprint Capacitor_SMD:C_0201_0603Metric -> Capacitor_SMD:C_0402_1005Metric; LCSC Part C47117441 -> C23733
- C4, C9: footprint Capacitor_SMD:C_0201_0603Metric -> Capacitor_SMD:C_0402_1005Metric; LCSC Part C307380 -> C1525
- C6: footprint Capacitor_SMD:C_0201_0603Metric -> Capacitor_SMD:C_0402_1005Metric; LCSC Part C272853 -> C15195
- L1: footprint Inductor_SMD:L_0201_0603Metric -> Inductor_SMD:L_0402_1005Metric; LCSC Part C86125 -> C18216
- L2: footprint Inductor_SMD:L_0201_0603Metric -> Inductor_SMD:L_0402_1005Metric; LCSC Part C49247134 -> C167472
- R1, R2, R3, R4, R5, R6: footprint Resistor_SMD:R_0201_0603Metric -> Resistor_SMD:R_0603_1608Metric
- R10, R11, R12, R7, R8, R9: footprint Resistor_SMD:R_0201_0603Metric -> Resistor_SMD:R_0603_1608Metric; LCSC Part C23345 -> C2907129
- R13: footprint Resistor_SMD:R_0201_0603Metric -> Resistor_SMD:R_0603_1608Metric; LCSC Part C2933227 -> C23065
Changed lines of the file:
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@@
 			)
 		)
-		(property "Footprint" "Capacitor_SMD:C_0201_0603Metric"
+		(property "Footprint" "Capacitor_SMD:C_0402_1005Metric"
 			(at 209.55 21.8948 0)
 			(hide yes)
@@
 			)
 		)
-		(property "LCSC Part" "C76935"
+		(property "LCSC Part" "C52923"
 			(at 205.74 22.86 90)
 			(hide yes)
@@
 			)
 		)
-		(property "Footprint" "Capacitor_SMD:C_0201_0603Metric"
+		(property "Footprint" "Capacitor_SMD:C_0402_1005Metric"
 			(at 171.1452 134.62 0)
 			(hide yes)
@@
 			)
 		)
-		(property "LCSC Part" "C76935"
+		(property "LCSC Part" "C52923"
 			(at 170.18 130.81 0)
 			(hide yes)
@@
 			)
 		)
-		(property "Footprint" "Resistor_SMD:R_0201_0603Metric"
+		(property "Footprint" "Resistor_SMD:R_0603_1608Metric"
 			(at 115.57 99.568 90)
 			(hide yes)
@@
 			)
 		)
-		(property "Footprint" "Capacitor_SMD:C_0201_0603Metric"
+		(property "Footprint" "Capacitor_SMD:C_0402_1005Metric"
 			(at 180.0352 39.37 0)
 			(hide yes)
@@
 			)
 		)
-		(property "LCSC Part" "C76935"
+		(property "LCSC Part" "C52923"
 			(at 179.07 35.56 0)
 			(hide yes)
@@
 			)
 		)
-		(property "Footprint" "Resistor_SMD:R_0201_0603Metric"
+		(property "Footprint" "Resistor_SMD:R_0603_1608Metric"
 			(at 115.57 124.968 90)
 			(hide yes)
@@
 			)
 		)
-		(property "Footprint" "Resistor_SMD:R_0201_0603Metric"
+		(property "Footprint" "Resistor_SMD:R_0603_1608Metric"
 			(at 242.57 89.662 90)
 			(hide yes)
@@
 			)
 		)
-		(property "LCSC Part" "C23345"
+		(property "LCSC Part" "C2907129"
 			(at 242.57 91.44 90)
 			(hide yes)
@@
 			)
 		)
-		(property "Footprint" "Resistor_SMD:R_0201_0603Metric"
+		(property "Footprint" "Resistor_SMD:R_0603_1608Metric"
 			(at 242.57 76.962 90)
 			(hide yes)
@@
 			)
 		)
-		(property "LCSC Part" "C23345"
+		(property "LCSC Part" "C2907129"
 			(at 242.57 78.74 90)
 			(hide yes)
@@
 			)
 		)
-		(property "Footprint" "Resistor_SMD:R_0201_0603Metric"
+		(property "Footprint" "Resistor_SMD:R_0603_1608Metric"
 			(at 242.57 79.502 90)
 			(hide yes)
@@
 			)
 		)
-		(property "LCSC Part" "C23345"
+		(property "LCSC Part" "C2907129"
 			(at 242.57 81.28 90)
 			(hide yes)
@@
 			)
 		)
-		(property "Footprint" "Capacitor_SMD:C_0201_0603Metric"
+		(property "Footprint" "Capacitor_SMD:C_0402_1005Metric"
 			(at 191.4652 39.37 0)
 			(hide yes)
@@
 			)
 		)
-		(property "LCSC Part" "C307380"
+		(property "LCSC Part" "C1525"
 			(at 190.5 35.56 0)
 			(hide yes)
@@
 			)
 		)
-		(property "Footprint" "Capacitor_SMD:C_0201_0603Metric"
+		(property "Footprint" "Capacitor_SMD:C_0402_1005Metric"
 			(at 173.6852 54.61 0)
 			(hide yes)
@@
 			)
 		)
-		(property "LCSC Part" "C76935"
+		(property "LCSC Part" "C52923"
 			(at 172.72 50.8 0)
 			(hide yes)
@@
 			)
 		)
-		(property "Footprint" "Inductor_SMD:L_0201_0603Metric"
+		(property "Footprint" "Inductor_SMD:L_0402_1005Metric"
 			(at 176.53 96.52 0)
 			(hide yes)
@@
 			)
 		)
-		(property "LCSC Part" "C49247134"
+		(property "LCSC Part" "C167472"
 			(at 176.53 96.52 90)
 			(hide yes)
@@
 			)
 		)
-		(property "Footprint" "Resistor_SMD:R_0201_0603Metric"
+		(property "Footprint" "Resistor_SMD:R_0603_1608Metric"
 			(at 158.242 154.94 90)
 			(hide yes)
@@
 			)
 		)
-		(property "Footprint" "Capacitor_SMD:C_0201_0603Metric"
+		(property "Footprint" "Capacitor_SMD:C_0402_1005Metric"
 			(at 256.2352 39.37 0)
 			(hide yes)
@@
 			)
 		)
-		(property "LCSC Part" "C76935"
+		(property "LCSC Part" "C52923"
 			(at 255.27 35.56 0)
 			(hide yes)
@@
 			)
 		)
-		(property "Footprint" "Capacitor_SMD:C_0201_0603Metric"
+		(property "Footprint" "Capacitor_SMD:C_0402_1005Metric"
 			(at 160.9852 54.61 0)
 			(hide yes)
@@
 			)
 		)
-		(property "LCSC Part" "C307380"
+		(property "LCSC Part" "C1525"
 			(at 160.02 50.8 0)
 			(hide yes)
@@
 			)
 		)
-		(property "Footprint" "Resistor_SMD:R_0201_0603Metric"
+		(property "Footprint" "Resistor_SMD:R_0603_1608Metric"
 			(at 76.708 46.99 90)
 			(hide yes)
@@
 			)
 		)
-		(property "Footprint" "Resistor_SMD:R_0201_0603Metric"
+		(property "Footprint" "Resistor_SMD:R_0603_1608Metric"
 			(at 242.57 84.582 90)
 			(hide yes)
@@
 			)
 		)
-		(property "LCSC Part" "C23345"
+		(property "LCSC Part" "C2907129"
 			(at 242.57 86.36 90)
 			(hide yes)
@@
 			)
 		)
-		(property "Footprint" "Resistor_SMD:R_0201_0603Metric"
+		(property "Footprint" "Resistor_SMD:R_0603_1608Metric"
 			(at 172.72 77.978 90)
 			(hide yes)
@@
 			)
 		)
-		(property "LCSC Part" "C2933227"
+		(property "LCSC Part" "C23065"
 			(at 172.72 76.2 90)
 			(hide yes)
@@
 			)
 		)
-		(property "Footprint" "Inductor_SMD:L_0201_0603Metric"
+		(property "Footprint" "Inductor_SMD:L_0402_1005Metric"
 			(at 167.64 46.99 0)
 			(hide yes)
@@
 			)
 		)
-		(property "LCSC Part" "C86125"
+		(property "LCSC Part" "C18216"
 			(at 167.64 46.99 90)
 			(hide yes)
@@
 			)
 		)
-		(property "Footprint" "Resistor_SMD:R_0201_0603Metric"
+		(property "Footprint" "Resistor_SMD:R_0603_1608Metric"
 			(at 242.57 87.122 90)
 			(hide yes)
@@
 			)
 		)
-		(property "LCSC Part" "C23345"
+		(property "LCSC Part" "C2907129"
 			(at 242.57 88.9 90)
 			(hide yes)
@@
 			)
 		)
-		(property "Footprint" "Resistor_SMD:R_0201_0603Metric"
+		(property "Footprint" "Resistor_SMD:R_0603_1608Metric"
 			(at 242.57 82.042 90)
 			(hide yes)
@@
 			)
 		)
-		(property "LCSC Part" "C23345"
+		(property "LCSC Part" "C2907129"
 			(at 242.57 83.82 90)
 			(hide yes)
@@
 			)
 		)
-		(property "Footprint" "Capacitor_SMD:C_0201_0603Metric"
+		(property "Footprint" "Capacitor_SMD:C_0402_1005Metric"
 			(at 240.9952 39.37 0)
 			(hide yes)
@@
 			)
 		)
-		(property "LCSC Part" "C272853"
+		(property "LCSC Part" "C15195"
 			(at 240.03 35.56 0)
 			(hide yes)
@@
 			)
 		)
-		(property "Footprint" "Resistor_SMD:R_0201_0603Metric"
+		(property "Footprint" "Resistor_SMD:R_0603_1608Metric"
 			(at 85.598 45.72 90)
 			(hide yes)
@@
 			)
 		)
-		(property "Footprint" "Capacitor_SMD:C_0201_0603Metric"
+		(property "Footprint" "Capacitor_SMD:C_0402_1005Metric"
 			(at 135.5852 49.53 0)
 			(hide yes)
@@
 			)
 		)
-		(property "LCSC Part" "C47117441"
+		(property "LCSC Part" "C23733"
 			(at 134.62 45.72 0)
 			(hide yes)
@@
 			)
 		)
-		(property "Footprint" "Resistor_SMD:R_0201_0603Metric"
+		(property "Footprint" "Resistor_SMD:R_0603_1608Metric"
 			(at 114.3 150.368 90)
 			(hide yes)

Commit message: Update project
Parts:
- C2: footprint Capacitor_SMD:C_0402_1005Metric -> Capacitor_SMD:C_0603_1608Metric; LCSC Part C23733 -> C69335
Changed lines of the file:
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@@
 			)
 		)
-		(property "Footprint" "Capacitor_SMD:C_0402_1005Metric"
+		(property "Footprint" "Capacitor_SMD:C_0603_1608Metric"
 			(at 135.5852 49.53 0)
 			(hide yes)
@@
 			)
 		)
-		(property "LCSC Part" "C23733"
+		(property "LCSC Part" "C69335"
 			(at 134.62 45.72 0)
 			(hide yes)

Commit message: Update project
Parts:
- C11, C12: value 10uF -> 10pF; LCSC Part C96446 -> C1634
Connections:
- net +3.3V: now also R4.1
- net GND: no longer R4.2
- net GPIO9: now also R4.2; no longer R4.1
Other:
- moved on the sheet: R4
Changed lines of the file:
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@@
 	)
 	(junction
+		(at 160.02 151.13)
+		(diameter 0)
+		(color 0 0 0 0)
+	)
+	(junction
 		(at 64.77 34.29)
 		(diameter 0)
@@
 	)
 	(junction
-		(at 160.02 151.13)
-		(diameter 0)
-		(color 0 0 0 0)
-	)
-	(junction
 		(at 100.33 41.91)
 		(diameter 0)
@@
 	(symbol
 		(lib_id "power:GND")
-		(at 160.02 158.75 0)
-		(unit 1)
-		(body_style 1)
-		(exclude_from_sim no)
-		(in_bom yes)
-		(on_board yes)
-		(in_pos_files yes)
-		(dnp no)
-		(fields_autoplaced yes)
-		(property "Reference" "#PWR024"
-			(at 160.02 165.1 0)
-			(hide yes)
-			(show_name no)
-			(do_not_autoplace no)
-			(effects
-				(font
-					(size 1.27 1.27)
-				)
-			)
-		)
-		(property "Value" "GND"
-			(at 160.02 163.83 0)
-			(show_name no)
-			(do_not_autoplace no)
-			(effects
-				(font
-					(size 1.27 1.27)
-				)
-			)
-		)
-		(property "Footprint" ""
-			(at 160.02 158.75 0)
-			(hide yes)
-			(show_name no)
-			(do_not_autoplace no)
-			(effects
-				(font
-					(size 1.27 1.27)
-				)
-			)
-		)
-		(property "Datasheet" ""
-			(at 160.02 158.75 0)
-			(hide yes)
-			(show_name no)
-			(do_not_autoplace no)
-			(effects
-				(font
-					(size 1.27 1.27)
-				)
-			)
-		)
-		(property "Description" "Power symbol creates a global label with name \"GND\" , ground"
-			(at 160.02 158.75 0)
-			(hide yes)
-			(show_name no)
-			(do_not_autoplace no)
-			(effects
-				(font
-					(size 1.27 1.27)
-				)
-			)
-		)
-		(pin "1"
-		)
-		(instances
-			(project "Devboard"
-				(path "/b2b70760-826f-4f05-b18d-4f006907a185"
-					(reference "#PWR024")
-					(unit 1)
-				)
-			)
-		)
-	)
-	(symbol
-		(lib_id "power:GND")
 		(at 96.52 102.87 0)
 		(unit 1)
@@
 			)
 		)
-		(property "Value" "10uF"
+		(property "Value" "10pF"
 			(at 171.45 104.1399 0)
 			(show_name no)
@@
 			)
 		)
-		(property "LCSC Part" "C96446"
+		(property "LCSC Part" "C1634"
 			(at 167.64 102.87 0)
 			(hide yes)
@@
 	(symbol
 		(lib_id "Device:R")
-		(at 160.02 154.94 0)
+		(at 160.02 147.32 0)
 		(unit 1)
 		(body_style 1)
@@
 		(in_pos_files yes)
 		(dnp no)
-		(fields_autoplaced yes)
 		(property "Reference" "R4"
-			(at 162.56 153.6699 0)
+			(at 155.194 146.05 0)
 			(show_name no)
 			(do_not_autoplace no)
@@
 		)
 		(property "Value" "10k"
-			(at 162.56 156.2099 0)
+			(at 155.194 148.59 0)
 			(show_name no)
 			(do_not_autoplace no)
@@
 		)
 		(property "Footprint" "Resistor_SMD:R_0603_1608Metric"
-			(at 158.242 154.94 90)
+			(at 158.242 147.32 90)
 			(hide yes)
 			(show_name no)
@@
 		)
 		(property "Datasheet" ""
-			(at 160.02 154.94 0)
+			(at 160.02 147.32 0)
 			(hide yes)
 			(show_name no)
@@
 		)
 		(property "Description" "Resistor"
-			(at 160.02 154.94 0)
+			(at 160.02 147.32 0)
 			(hide yes)
 			(show_name no)
@@
 		)
 		(property "LCSC Part" "C2930027"
-			(at 160.02 154.94 0)
+			(at 160.02 147.32 0)
 			(hide yes)
 			(show_name no)
@@
 		)
 		(property "KLC_S3.3" ""
-			(at 160.02 154.94 0)
+			(at 160.02 147.32 0)
 			(hide yes)
 			(show_name no)
@@
 		)
 		(property "KLC_S4.1" ""
-			(at 160.02 154.94 0)
+			(at 160.02 147.32 0)
 			(hide yes)
 			(show_name no)
@@
 			)
 		)
-		(property "Value" "10uF"
+		(property "Value" "10pF"
 			(at 156.21 104.1399 0)
 			(show_name no)
@@
 			)
 		)
-		(property "LCSC Part" "C96446"
+		(property "LCSC Part" "C1634"
 			(at 152.4 102.87 0)
 			(hide yes)
@@
 					(unit 1)
 				)
+			)
+		)
+	)
+	(symbol
+		(lib_id "power:+3.3V")
+		(at 160.02 143.51 0)
+		(unit 1)
+		(body_style 1)
+		(exclude_from_sim no)
+		(in_bom yes)
+		(on_board yes)
+		(in_pos_files yes)
+		(dnp no)
+		(fields_autoplaced yes)
+		(property "Reference" "#PWR011"
+			(at 160.02 147.32 0)
+			(hide yes)
+			(show_name no)
+			(do_not_autoplace no)
+			(effects
+				(font
+					(size 1.27 1.27)
+				)
+			)
+		)
+		(property "Value" "+3.3V"
+			(at 160.02 138.43 0)
+			(show_name no)
+			(do_not_autoplace no)
+			(effects
+				(font
+					(size 1.27 1.27)
+				)
+			)
+		)
+		(property "Footprint" ""
+			(at 160.02 143.51 0)
+			(hide yes)
+			(show_name no)
+			(do_not_autoplace no)
+			(effects
+				(font
+					(size 1.27 1.27)
+				)
+			)
+		)
+		(property "Datasheet" ""
+			(at 160.02 143.51 0)
+			(hide yes)
+			(show_name no)
+			(do_not_autoplace no)
+			(effects
+				(font
+					(size 1.27 1.27)
+				)
+			)
+		)
+		(property "Description" "Power symbol creates a global label with name \"+3.3V\""
+			(at 160.02 143.51 0)
+			(hide yes)
+			(show_name no)
+			(do_not_autoplace no)
+			(effects
+				(font
+					(size 1.27 1.27)
+				)
+			)
+		)
+		(pin "1"
+		)
+		(instances
+			(project "Devboard"
+				(path "/b2b70760-826f-4f05-b18d-4f006907a185"
+					(reference "#PWR011")
+					(unit 1)
+				)
